File: codepad.kicad_pcb (KiCad board)
At the start: 2 copper layers, 4.4 x 4.3 mm, 39 parts, among them SW1 SW_Push, SW2 SW_Push, SW3 SW_Push, SW4 SW_Push, SW5 SW_Push, SW6 SW_Push, SW7 SW_Push, SW8 SW_Push, SW9 RotaryEncoder_Switch, U1 MOUDLE-SEEEDUINO-XIAO, U2 ER_OLEDM0.91_1x-I2C

Commit message: restart
working from start after watchinh a tutorial
Parts:
- removed D10, D11, D12, D13, D14, D15, D16, D17, D18, D19, D20, D21, D22, D23, D24, D25, D26, D27, D28: SK6812MINI-E, hackclub:SK6812MINI-E_fixed
- moved D9 61.7 mm to (100.4, 73.5)
- moved D1 60.3 mm to (100.7, 112.5)
- moved SW7 54.9 mm to (68.0, 78.0)
- moved SW8 54.9 mm to (87.5, 78.0)
- moved U1 51.4 mm to (74.1, 52.7)
- moved D6 50.8 mm to (100.2, 92.5)
- moved SW3 46.4 mm to (68.0, 117.0)
- moved D8 43.7 mm to (79.9, 73.5)
- moved D2 42.1 mm to (80.5, 112.5)
- moved SW1 41.1 mm to (107.0, 117.0)
- moved SW4 40.5 mm to (68.0, 97.4)
- moved SW9 35.3 mm to (129.5, 56.0), turned to -90 degrees
- moved D5 30.8 mm to (80.5, 93.0)
- moved D7 30.1 mm to (60.7, 73.5)
- moved D3 27.7 mm to (61.4, 112.5)
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Connections:
- D1 pad 1: Net-(D1-K) -> row 2
- D2 pad 1: Net-(D1-K) -> row 2
- D3 pad 1: Net-(D1-K) -> row 2
- D4 pad 1: Net-(D4-K) -> row 1
- D5 pad 1: Net-(D4-K) -> row 1
- D6 pad 1: Net-(D4-K) -> row 1
- D7 pad 1: Net-(D7-K) -> row 0
- D8 pad 1: Net-(D7-K) -> row 0
- D9 pad 1: Net-(D7-K) -> row 0
- SW1 pad 1: Net-(D7-A) -> Net-(D1-A)
- SW1 pad 2: Net-(SW1-Pad2) -> column 0
- SW2 pad 1: Net-(D8-A) -> Net-(D2-A)
- SW2 pad 2: Net-(SW2-Pad2) -> column 1
- SW3 pad 1: Net-(D4-A) -> Net-(D3-A)
- SW3 pad 2: Net-(SW1-Pad2) -> column 2
- SW4 pad 1: Net-(D5-A) -> Net-(D4-A)
- SW4 pad 2: Net-(SW2-Pad2) -> column 0
- SW5 pad 1: Net-(D1-A) -> Net-(D5-A)
- SW5 pad 2: Net-(SW1-Pad2) -> column 1
- SW6 pad 1: Net-(D2-A) -> Net-(D6-A)
- SW6 pad 2: Net-(SW2-Pad2) -> column 2
- SW7 pad 1: Net-(D6-A) -> Net-(D7-A)
- SW7 pad 2: Net-(SW7-Pad2) -> column 0
- SW8 pad 1: Net-(D3-A) -> Net-(D8-A)
- SW8 pad 2: Net-(SW7-Pad2) -> column 1
- SW9 pad A: Net-(U1-PA4_A1_D1) -> Net-(U1-PB08_A6_D6_TX)
- SW9 pad B: Net-(U1-PA10_A2_D2) -> Net-(U1-PA11_A3_D3)
- SW9 pad S1: Net-(SW7-Pad2) -> Net-(D9-A)
- SW9 pad S2: Net-(D9-A) -> column 2
- U1 pad 1: Net-(D20-DIN) -> column 0
- U1 pad 10: unconnected-(U1-PA5_A9_D9_MISO-Pad10) -> row 1
- U1 pad 11: unconnected-(U1-PA6_A10_D10_MOSI-Pad11) -> row 2
- U1 pad 12: unconnected-(U1-3V3-Pad12) -> 3.3v
- U1 pad 14: Net-(D17-VDD) -> unconnected-(U1-5V-Pad14)
- U1 pad 2: Net-(U1-PA4_A1_D1) -> column 1
- U1 pad 3: Net-(U1-PA10_A2_D2) -> column 2
- U1 pad 4: unconnected-(U1-PA11_A3_D3-Pad4) -> Net-(U1-PA11_A3_D3)
- U1 pad 7: unconnected-(U1-PB08_A6_D6_TX-Pad7) -> Net-(U1-PB08_A6_D6_TX)
- U1 pad 9: unconnected-(U1-PA7_A8_D8_SCK-Pad9) -> row 0
- U2 pad 2: unconnected-(U2-VCC-Pad2) -> 3.3v
Routing:
- net row 2: track 0.00 -> 124.1 mm
- net Net-(D17-VDD): track 106.6 -> 0.00 mm
- net Net-(D17-VSS): track 103.4 -> 0.00 mm
- net row 1: track 0.00 -> 89.5 mm
- net Net-(U1-PA8_A4_D4_SDA): track 69.2 -> 0.00 mm
- net Net-(U1-PA9_A5_D5_SCL): track 65.3 -> 0.00 mm
- net row 0: track 0.00 -> 62.7 mm
- net Net-(U1-PA4_A1_D1): track 57.1 -> 0.00 mm
- net Net-(U1-PA10_A2_D2): track 48.4 -> 0.00 mm
- net unconnected-(D19-DOUT-Pad4): track 37.9 -> 0.00 mm
- net Net-(D20-DIN): track 37.9 -> 0.00 mm
- net Net-(D21-DOUT): track 13.2 -> 0.00 mm
- net Net-(D22-DOUT): track 11.7 -> 0.00 mm
- net Net-(D17-DOUT): track 11.3 -> 0.00 mm
- net Net-(D18-DOUT): track 10.3 -> 0.00 mm
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Other:
- board outline removed
